File: 01 - Avionics 25-26/Upper Bulkhead Connection Revision A/Upper_Bulkhead_Connection_Rev_A.kicad_sch (KiCad schematic)
At the start: 2 parts, among them J1 2601-3108, J2 M12A-08PMMP-SF8001

Commit message: Add files via upload
Other:
- note added: "M12_7 -- TeleMetrumV4 Apogee+ (TMD+) -- 2601_3108_13&14"
- note added: "M12_8 -- TeleMetrumV4 Apogee- (TMD-) -- 2601_3108_15&16"
- note removed: "M12_7 -- TeleMetrumV4 Apogee+ (TMA+) -- 2601_3108_13&14"
- note removed: "M12_8 -- TeleMetrumV4 Apogee- (TMA-) -- 2601_3108_15&16"
Changed lines of the file:
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@@
 		)
 	)
-	(text "M12_8 -- TeleMetrumV4 Apogee- (TMA-) -- 2601_3108_15&16"
+	(text "M12_8 -- TeleMetrumV4 Apogee- (TMD-) -- 2601_3108_15&16"
 		(exclude_from_sim no)
 		(at 94.488 75.692 0)
@@
 		)
 	)
-	(text "M12_7 -- TeleMetrumV4 Apogee+ (TMA+) -- 2601_3108_13&14"
+	(text "M12_7 -- TeleMetrumV4 Apogee+ (TMD+) -- 2601_3108_13&14"
 		(exclude_from_sim no)
 		(at 94.488 73.406 0)

Commit message: Add files via upload
Connections:
- net at J1.1 (1_1), J1.2 (1_2): now also J2.6; no longer J2.1
- net at J1.3 (2_1), J1.4 (2_2): now also J2.7; no longer J2.2
- net at J1.5 (3_1), J1.6 (3_2): now also J2.1; no longer J2.3
- net at J1.7 (4_1), J1.8 (4_2): now also J2.8; no longer J2.4
- net at J1.10 (5_2), J1.9 (5_1): now also J2.2; no longer J2.5
- net at J1.11 (6_1), J1.12 (6_2): now also J2.3; no longer J2.6
- net at J1.13 (7_1), J1.14 (7_2): now also J2.4; no longer J2.7
- net at J1.15 (8_1), J1.16 (8_2): now also J2.5; no longer J2.8
Other:
- note added: "M12_1 -- Blue Raven Apo+ (BRD+) -- 2601_3108_5&6"
- note added: "M12_2 -- TeleMetrumV4 Main+ (TMM+) -- 2601_3108_9&10"
- note added: "M12_3 -- TeleMetrumV4 Main- (TMM-) -- 2601_3108_11&12"
- note added: "M12_4 -- TeleMetrumV4 Apogee+ (TMD+) -- 2601_3108_13&14"
- note added: "M12_5 -- TeleMetrumV4 Apogee- (TMD-) -- 2601_3108_15&16"
- note added: "M12_6 -- Blue Raven Main+ (BRM+) -- 2601_3108_1&2"
- note added: "M12_7 -- Blue Raven Main- (BRM-) -- 2601_3108_3&4"
- note added: "M12_8 -- Blue Raven Apo (BRD-) -- 2601_3108_7&8"
- note removed: "M12_1 -- Blue Raven Main+ (BRM+) -- 2601_3108_1&2"
- note removed: "M12_2 -- Blue Raven Main- (BRM-) -- 2601_3108_3&4"
- note removed: "M12_3 -- Blue Raven Apo+ (BRD+) -- 2601_3108_5&6"
- note removed: "M12_4 -- Blue Raven Apo (BRD-) -- 2601_3108_7&8"
- note removed: "M12_5 -- TeleMetrumV4 Main+ (TMM+) -- 2601_3108_9&10"
- note removed: "M12_6 -- TeleMetrumV4 Main- (TMM-) -- 2601_3108_11&12"
- note removed: "M12_7 -- TeleMetrumV4 Apogee+ (TMD+) -- 2601_3108_13&14"
- note removed: "M12_8 -- TeleMetrumV4 Apogee- (TMD-) -- 2601_3108_15&16"
