File: 01 - Avionics 25-26/Upper Bulkhead Connection Revision A/Upper_Bulkhead_Connection_Rev_A.kicad_pcb (KiCad board)
At the start: 2 copper layers, 38 x 40.9 mm, 4 parts, among them J1 2601-3108, J2 M12A-08PMMP-SF8001

Commit message: Add files via upload
Other:
- board text added: "TMD+"
- board text added: "TMD-"
Changed lines of the file:
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@@
 		)
 	)
-	(gr_text "TMA-"
+	(gr_text "TMD-"
 		(at 98.5 108.5 0)
 		(layer "F.SilkS")
@@
 		)
 	)
-	(gr_text "TMA+"
+	(gr_text "TMD+"
 		(at 105 101 0)
 		(layer "F.SilkS")
@@
 		)
 	)
-	(gr_text "TMA-"
-		(at 102.5 108.5 -0)
-		(layer "B.SilkS")
-		(effects
-			(font
-				(size 1 1)
-				(thickness 0.2)
-				(bold yes)
-			)
-			(justify left bottom mirror)
-		)
-	)
-	(gr_text "TMA+"
-		(at 109 101 -0)
-		(layer "B.SilkS")
-		(effects
+	(gr_text "TMD-"
+		(at 102.5 108.5 0)
+		(layer "B.SilkS")
+		(effects
+			(font
+				(size 1 1)
+				(thickness 0.2)
+				(bold yes)
+			)
+			(justify left bottom mirror)
+		)
+	)
+	(gr_text "TMD+"
+		(at 109 101 0)
+		(layer "B.SilkS")
+		(effects

Commit message: Add files via upload
Parts:
- J2: moved to B.Cu
- moved J1 6.00 mm to (88.0, 79.0)
- moved REF** 6.00 mm to (86.0, 99.5)
- moved REF** 6.00 mm to (114.0, 99.5)
Routing:
- net Net-(J1-7_1): track 19.0 -> 26.1 mm
- net Net-(J1-6_1): track 22.3 -> 28.5 mm
- net Net-(J1-5_1): track 25.6 -> 31.4 mm
- net Net-(J1-1_1): track 27.9 -> 23.1 mm
- net Net-(J1-2_1): track 18.8 -> 22.5 mm
- net Net-(J1-8_1): track 27.4 -> 26.3 mm
- net Net-(J1-3_1): track 22.5 -> 23.4 mm
Other:
- board text added: "${REFERENCE}"
- board text removed: "TMD+"
- board text removed: "TMD-"

Commit message: Add files via upload
Parts:
- moved REF** 0.50 mm to (86.0, 100.0)
- moved REF** 0.50 mm to (114.0, 100.0)
Other:
- board size 38 x 40.9 mm -> 40 x 42.6 mm
Changed lines of the file:
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@@
 	(footprint "MountingHole:MountingHole_3.2mm_M3"
 		(layer "F.Cu")
-		(at 86 99.5)
+		(at 86 100)
 		(descr "Mounting Hole 3.2mm, M3, no annular, generated by kicad-footprint-generator mountinghole.py")
 		(tags "mountinghole M3")
@@
 	(footprint "MountingHole:MountingHole_3.2mm_M3"
 		(layer "F.Cu")
-		(at 114 99.5)
+		(at 114 100)
 		(descr "Mounting Hole 3.2mm, M3, no annular, generated by kicad-footprint-generator mountinghole.py")
 		(tags "mountinghole M3")
@@
 	(gr_line
 		(start 84 86)
-		(end 81 100)
+		(end 80 100)
 		(stroke
 			(width 0.2)
@@
 	)
 	(gr_arc
-		(start 119 100)
-		(mid 100 113.924859)
-		(end 81 100.000001)
+		(start 119.999999 100.000001)
+		(mid 100 115.615527)
+		(end 80.000001 100)
 		(stroke
 			(width 0.05)
-			(type default)
+			(type solid)
 		)
 		(layer "Edge.Cuts")
@@
 	)
 	(gr_line
-		(start 119 100)
+		(start 120 100)
 		(end 116 86)
 		(stroke
@@
 	)
 	(gr_text "${REFERENCE}"
-		(at 86 99.5 0)
+		(at 100.300001 81.5 0)
 		(layer "F.Fab")
 		(effects
@@
 	)
 	(gr_text "${REFERENCE}"
-		(at 100.300001 81.5 0)
+		(at 86 99.5 0)
 		(layer "F.Fab")
 		(effects

Commit message: Add files via upload
Other:
- board text added: "TMD+"
- board text added: "TMD-"
- board text removed: "TMA+"
- board text removed: "TMA-"
Changed lines of the file:
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@@
 		(layer "Edge.Cuts")
 	)
-	(gr_text "TMA+"
+	(gr_text "TMD+"
 		(at 109.5 91 90)
 		(layer "F.SilkS")
@@
 		)
 	)
-	(gr_text "TMA-"
-		(at 113 91 90)
+	(gr_text "TMD-"
+		(at 113.25 91 90)
 		(layer "F.SilkS")
 		(effects
@@
 		)
 	)
-	(gr_text "TMA-"
+	(gr_text "TMD-"
 		(at 100.25 99.5 90)
 		(layer "F.SilkS")
@@
 		)
 	)
-	(gr_text "TMA+"
+	(gr_text "TMD+"
 		(at 96 102 90)
 		(layer "F.SilkS")
@@
 		)
 	)
-	(gr_text "TMA+"
-		(at 108.5 91 -90)
-		(layer "B.SilkS")
-		(effects
-			(font
-				(size 1 1)
-				(thickness 0.2)
-				(bold yes)
-			)
-			(justify left bottom mirror)
-		)
-	)
-	(gr_text "TMA-"
-		(at 112 91 -90)
-		(layer "B.SilkS")
-		(effects
-			(font
-				(size 1 1)
-				(thickness 0.2)
-				(bold yes)
-			)
-			(justify left bottom mirror)
-		)
-	)
-	(gr_text "TMA-"
-		(at 99 99.5 -90)
+	(gr_text "TMD+"
+		(at 108.5 91 270)
+		(layer "B.SilkS")
+		(effects
+			(font
+				(size 1 1)
+				(thickness 0.2)
+				(bold yes)
+			)
+			(justify left bottom mirror)
+		)
+	)
+	(gr_text "TMD-"
+		(at 112 91 270)
+		(layer "B.SilkS")
+		(effects
+			(font
+				(size 1 1)
+				(thickness 0.2)
+				(bold yes)
+			)
+			(justify left bottom mirror)
+		)
+	)
+	(gr_text "TMD-"
+		(at 99 99.5 270)
 		(layer "B.SilkS")
 		(effects
@@
 		)
 	)
-	(gr_text "TMA+"
-		(at 94.75 102 -90)
-		(layer "B.SilkS")
-		(effects
+	(gr_text "TMD+"
+		(at 94.75 102 270)
+		(layer "B.SilkS")
+		(effects

Commit message: Add files via upload
Connections:
- J2 pad 1: Net-(J1-1_1) -> Net-(J1-3_1)
- J2 pad 2: Net-(J1-2_1) -> Net-(J1-5_1)
- J2 pad 3: Net-(J1-3_1) -> Net-(J1-6_1)
- J2 pad 4: Net-(J1-4_1) -> Net-(J1-7_1)
- J2 pad 5: Net-(J1-5_1) -> Net-(J1-8_1)
- J2 pad 6: Net-(J1-6_1) -> Net-(J1-1_1)
- J2 pad 7: Net-(J1-7_1) -> Net-(J1-2_1)
- J2 pad 8: Net-(J1-8_1) -> Net-(J1-4_1)
Routing:
- net Net-(J1-5_1): track 31.4 -> 20.1 mm
- net Net-(J1-6_1): track 28.5 -> 21.4 mm
- net Net-(J1-8_1): track 26.3 -> 31.7 mm
- net Net-(J1-1_1): track 23.1 -> 27.8 mm
- net Net-(J1-4_1): track 25.4 -> 21.6 mm
- net Net-(J1-7_1): track 26.1 -> 28.9 mm
- net Net-(J1-3_1): track 23.4 -> 21.3 mm
- net Net-(J1-2_1): track 22.5 -> 23.4 mm
Other:
- board text removed: "${REFERENCE}"

Commit message: Add files via upload
Parts:
- added G***: LOGO, Logos:MST_RDT_Rocket_Logo, F.Cu at (110.0, 107.0)
- added G***: LOGO, Logos:MST_RDT_Rocket_Logo, B.Cu at (90.0, 107.0)
Other:
- board text added: "MST RDT"
- board text added: "SINE LABORE NIHIL"
