File: 01 - Avionics 25-26/SRAD FC Rev B/KiCAD Files/GPS.kicad_sch (KiCad schematic)
At the start: 0 parts

Commit message: Added GPS schematic
Added GPS schematic
Parts:
- added C1, C2: 100n, Resistor_SMD:R_0603_1608Metric, symbol Device:C_Small
- added GPS: SAM-M10Q-00B, GPS_SAM_M10Q_00B:XCVR_SAM-M10Q-00B, symbol SAM-M10Q-00B:SAM-M10Q-00B
Connections:
- new net +3.3V: C1.2, C2.2, GPS.17 (VCC), GPS.2 (V_IO)
- new net EXTINT: GPS.19 (EXTINT)
- new net GND: C1.1, C2.1, GPS.1 (GND), GPS.10 (GND__4), GPS.11 (GND__5), GPS.15 (GND__6), GPS.16 (GND__7), GPS.20 (GND__8), GPS.4 (GND__1), GPS.5 (GND__2), GPS.6 (GND__3)
- new net RESET: GPS.18 (~{RESET})
- new net RXD: GPS.14 (RXD)
- new net SAFEBOOT: GPS.8 (~{SAFEBOOT})
- new net TIMEPULSE: GPS.7 (TIMEPULSE)
- new net TXD: GPS.13 (TXD)
- no-connect marks 0 -> 3

Commit message: Adjusted annotations and named the microcontroller reference
Parts:
- renumbered GPS to GPS1
Changed lines of the file:
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@@
 		(dnp no)
 		(fields_autoplaced yes)
-		(property "Reference" "GPS"
+		(property "Reference" "GPS1"
 			(at 139.7 67.31 0)
 			(effects
@@
 			(project "SRAD FC Rev B"
 				(path "/1dd9e63a-24f2-43c6-ae21-66b89e6998f2/b03efcbd-12ef-4a08-953b-a02584827ea7"
-					(reference "GPS")
+					(reference "GPS1")
 					(unit 1)
 				)

Commit message: GPS footprint and symbol library update
Parts:
- GPS1: footprint GPS_SAM_M10Q_00B:XCVR_SAM-M10Q-00B -> SAM_M10Q_00B:XCVR_SAM-M10Q-00B
Changed lines of the file:
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@@
 			)
 		)
-		(property "Footprint" "GPS_SAM_M10Q_00B:XCVR_SAM-M10Q-00B"
+		(property "Footprint" "SAM_M10Q_00B:XCVR_SAM-M10Q-00B"
 			(at 139.7 90.17 0)
 			(effects

Commit message: made changes to microcontroller and GPS. GPS footprint needs to be fixed and assigned again
Parts:
- GPS1: footprint SAM_M10Q_00B:XCVR_SAM-M10Q-00B -> Package_LGA:ublox_LGA-53_4.5x4.5mm_Layout9x9_P0.5mm
Changed lines of the file:
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@@
 			)
 		)
-		(property "Footprint" "SAM_M10Q_00B:XCVR_SAM-M10Q-00B"
+		(property "Footprint" "Package_LGA:ublox_LGA-53_4.5x4.5mm_Layout9x9_P0.5mm"
 			(at 139.7 90.17 0)
 			(effects

Commit message: added power as hierarchical sheet pins
Connections:
- net +3.3V renamed GPS_3.3V_POWER
Changed lines of the file:
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@@
+		)
+	)
+	(hierarchical_label "GPS_3.3V_POWER"
+		(shape output)
+		(at 189.23 57.15 90)
+		(effects
+			(font
+				(size 1.27 1.27)
+			)
+			(justify left)
 		)
 	)
@@
 					(unit 1)
 				)
-			)
-		)
-	)
-	(symbol
-		(lib_id "power:+3.3V")
-		(at 189.23 57.15 0)
-		(unit 1)
-		(exclude_from_sim no)
-		(in_bom yes)
-		(on_board yes)
-		(dnp no)
-		(property "Reference" "#PWR03"
-			(at 189.23 60.96 0)
-			(effects
-				(font
-					(size 1.27 1.27)
-				)
-				(hide yes)
-			)
-		)
-		(property "Value" "+3.3V"
-			(at 189.23 53.34 0)
-			(effects
-				(font
-					(size 1.27 1.27)
-				)
-			)
-		)
-		(property "Footprint" ""
-			(at 189.23 57.15 0)
-			(effects
-				(font
-					(size 1.27 1.27)
-				)
-				(hide yes)
-			)
-		)
-		(property "Datasheet" ""
-			(at 189.23 57.15 0)
-			(effects
-				(font
-					(size 1.27 1.27)
-				)
-				(hide yes)
-			)
-		)
-		(property "Description" ""
-			(at 189.23 57.15 0)
-			(effects
-				(font
-					(size 1.27 1.27)
-				)
-				(hide yes)
-			)
-		)
-		(pin "1"
-		)
-		(instances
-			(project "SRAD FC Rev B"
-				(path "/1dd9e63a-24f2-43c6-ae21-66b89e6998f2/b03efcbd-12ef-4a08-953b-a02584827ea7"
-					(reference "#PWR03")
-					(unit 1)
-				)

Commit message: fixed some library symbold
Parts:
- removed GPS1: SAM-M10Q-00B, Package_LGA:ublox_LGA-53_4.5x4.5mm_Layout9x9_P0.5mm, symbol SAM-M10Q-00B:SAM-M10Q-00B
- added U3: SAM-M10Q-00B, SAM_M10Q_00B:SAM-M10Q_UBL, symbol SAM-M10Q-00B:SAM-M10Q-00B
Connections:
- net EXTINT: now also U3.19 (EXTINT)
- net GND: now also U3.1 (GND), U3.10 (GND), U3.11 (GND), U3.15 (GND), U3.16 (GND), U3.20 (GND), U3.4 (GND), U3.5 (GND), U3.6 (GND)
- net GPS_3.3V_POWER: now also U3.2 (V_IO), U3.3 (V_BCKP)
- net RESET: now also U3.18 (RESET_N)
- net RXD: now also U3.14 (RXD)
- net SAFEBOOT: now also U3.8 (SAFEBOOT_N)
- net TIMEPULSE: now also U3.7 (TIMEPULSE)
- net TXD: now also U3.13 (TXD)
- no-connect marks 3 -> 0
Other:
- moved on the sheet: C1, C2

Commit message: more changes based on seth's feedback
Connections:
- net GPS_3.3V_POWER: now also U3.17 (VCC); no longer U3.3 (V_BCKP)
Changed lines of the file:
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@@
+	)
+	(junction
+		(at 73.66 60.96)
+		(diameter 0)
+		(color 0 0 0 0)
 	)
 	(junction
@@
 	)
 	(junction
-		(at 107.95 85.09)
-		(diameter 0)
-		(color 0 0 0 0)
-	)
-	(junction
 		(at 186.69 92.71)
 		(diameter 0)
@@
 	(wire
 		(pts
-			(xy 73.66 85.09) (xy 107.95 85.09)
-		)
-		(stroke
-			(width 0)
-			(type default)
-		)
-	)
-	(wire
-		(pts
 			(xy 172.72 97.79) (xy 187.96 97.79)
 		)
@@
 	(wire
 		(pts
-			(xy 107.95 85.09) (xy 111.76 85.09)
+			(xy 242.57 90.17) (xy 172.72 90.17)
+		)
+		(stroke
+			(width 0)
+			(type default)
+		)
+	)
+	(wire
+		(pts
+			(xy 242.57 60.96) (xy 242.57 90.17)
+		)
+		(stroke
+			(width 0)
+			(type default)
+		)
+	)
+	(wire
+		(pts
+			(xy 73.66 85.09) (xy 111.76 85.09)
 		)
 		(stroke
@@
 	(wire
 		(pts
-			(xy 107.95 87.63) (xy 111.76 87.63)
-		)
-		(stroke
-			(width 0)
-			(type default)
-		)
-	)
-	(wire
-		(pts
 			(xy 86.36 95.25) (xy 97.79 95.25)
 		)
@@
 	(wire
 		(pts
+			(xy 73.66 60.96) (xy 242.57 60.96)
+		)
+		(stroke
+			(width 0)
+			(type default)
+		)
+	)
+	(wire
+		(pts
 			(xy 203.2 87.63) (xy 172.72 87.63)
 		)
@@
 		)
 		(stroke
-			(width 0)
-			(type default)
-		)
-	)
-	(wire
-		(pts
-			(xy 107.95 85.09) (xy 107.95 87.63)
-		)
-		(stroke
