File: 01 - Avionics 25-26/SRAD FC Rev B/KiCAD Files/High G Accelerometer.kicad_sch (KiCad schematic)
At the start: 0 parts

Commit message: High G Accelerometer accelerometer schematic
Parts:
- added C15, C16: 0.1uF, symbol Device:C_Small
- added U2: ADXL372BCCZ-RL7, ADXL372BCCZ-RL7:PQFN50P322X300X114-16N, symbol ADXL372BCCZ-RL7:ADXL372BCCZ-RL7
Connections:
- new net ACCEL_INT1: U2.11 (INT1)
- new net ACCEL_INT2: U2.9 (INT2)
- new net ACCEL_SPI_CS: U2.8 (~{CS}/SCL)
- new net ACCEL_SPI_MISO: U2.7 (MISO)
- new net ACCEL_SPI_MOSI: U2.6 (MOSI/SDA)
- new net ACCEL_SPI_SCLK: U2.4 (SCLK)
- new net ACCEL_VDD_IO: C16.2, U2.1 (VDDI/O)
- new net ACCEL_VS: C15.2, U2.14 (VS)
- new net GND: C15.1, C16.1, U2.12 (GND), U2.13 (GND__1), U2.16 (GND__2)

Commit message: moved..... stuff
Connections:
- net ACCEL_VDD_IO renamed +3.3V
- net ACCEL_VS renamed +2.5V
Changed lines of the file:
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@@
 		(comment 1 "Author(s): Adam Seals")
+	)
+	(text_box "Vs is sensitive to noise. Increased noise will increase measurement error. If Vs and Vdd i/o share the same source, it can lead to clock noise on the Vs line. If we are stuck with a noisy voltage source for Vs then there are things we can do in the accelerometer schematic to mitigate the issue.\n\nAdditionally, Vs prefers to be at 2.5v, although it will function between 1.6v and 3.3v."
+		(exclude_from_sim no)
+		(at 137.16 116.84 0)
+		(size 34.29 30.48)
+		(margins 0.9525 0.9525 0.9525 0.9525)
+		(stroke
+			(width 0)
+			(type solid)
+		)
+		(fill
+			(type none)
+		)
+		(effects
+			(font
+				(size 1.27 1.27)
+			)
+			(justify left top)
+		)
 	)
 	(junction
@@
 		)
 	)
-	(hierarchical_label "ACCEL_VDD_IO"
-		(shape input)
-		(at 185.42 85.09 0)
-		(effects
-			(font
-				(size 1.27 1.27)
-			)
-			(justify left)
-		)
-	)
 	(hierarchical_label "ACCEL_SPI_CS"
 		(shape input)
@@
 			)
 			(justify right)
-		)
-	)
-	(hierarchical_label "ACCEL_VS"
-		(shape input)
-		(at 185.42 82.55 0)
-		(effects
-			(font
-				(size 1.27 1.27)
-			)
-			(justify left)
 		)
 	)
@@
 	)
 	(symbol
+		(lib_id "power:+3.3V")
+		(at 185.42 85.09 270)
+		(unit 1)
+		(exclude_from_sim no)
+		(in_bom yes)
+		(on_board yes)
+		(dnp no)
+		(fields_autoplaced yes)
+		(property "Reference" "#PWR027"
+			(at 181.61 85.09 0)
+			(effects
+				(font
+					(size 1.27 1.27)
+				)
+				(hide yes)
+			)
+		)
+		(property "Value" "+3.3V"
+			(at 189.23 85.0899 90)
+			(effects
+				(font
+					(size 1.27 1.27)
+				)
+				(justify left)
+			)
+		)
+		(property "Footprint" ""
+			(at 185.42 85.09 0)
+			(effects
+				(font
+					(size 1.27 1.27)
+				)
+				(hide yes)
+			)
+		)
+		(property "Datasheet" ""
+			(at 185.42 85.09 0)
+			(effects
+				(font
+					(size 1.27 1.27)
+				)
+				(hide yes)
+			)
+		)
+		(property "Description" "Power symbol creates a global label with name \"+3.3V\""
+			(at 185.42 85.09 0)
+			(effects
+				(font
+					(size 1.27 1.27)
+				)
+				(hide yes)
+			)
+		)
+		(pin "1"
+		)
+		(instances
+			(project "SRAD FC Rev B"
+				(path "/1dd9e63a-24f2-43c6-ae21-66b89e6998f2/a64879cb-ca83-46f5-8e0d-bba02df69177"
+					(reference "#PWR027")
+					(unit 1)
+				)
+			)
+		)
+	)
+	(symbol
 		(lib_id "Device:C_Small")
 		(at 179.07 74.93 0)
@@
 					(unit 1)
 				)
+			)
+		)
+	)
+	(symbol
+		(lib_id "power:+3.3V")
+		(at 185.42 82.55 270)
+		(unit 1)
+		(exclude_from_sim no)
+		(in_bom yes)
+		(on_board yes)
+		(dnp no)
+		(fields_autoplaced yes)
+		(property "Reference" "#PWR026"
+			(at 181.61 82.55 0)
+			(effects
+				(font
+					(size 1.27 1.27)
+				)
+				(hide yes)
+			)
+		)
+		(property "Value" "+2.5V"
+			(at 189.23 82.5499 90)
+			(effects
+				(font
+					(size 1.27 1.27)
+				)
+				(justify left)
+			)
+		)
+		(property "Footprint" ""
+			(at 185.42 82.55 0)
+			(effects
+				(font
+					(size 1.27 1.27)
+				)
+				(hide yes)
+			)
+		)
+		(property "Datasheet" ""
+			(at 185.42 82.55 0)
+			(effects
+				(font
+					(size 1.27 1.27)
+				)
+				(hide yes)
+			)
+		)
+		(property "Description" "Power symbol creates a global label with name \"+1.8V\""
+			(at 185.42 82.55 0)
+			(effects
+				(font
+					(size 1.27 1.27)
+				)
+				(hide yes)
+			)
+		)
+		(pin "1"
+		)
+		(instances
+			(project "SRAD FC Rev B"
+				(path "/1dd9e63a-24f2-43c6-ae21-66b89e6998f2/a64879cb-ca83-46f5-8e0d-bba02df69177"
+					(reference "#PWR026")
+					(unit 1)
+				)

Commit message: added power as hierarchical sheet pins
Connections:
- net +2.5V renamed ACCEL_2.5V_POWER_SENSITIVE
- net +3.3V renamed ACCEL_3.3V_POWER
Changed lines of the file:
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@@
+		)
+	)
+	(hierarchical_label "ACCEL_3.3V_POWER"
+		(shape input)
+		(at 185.42 85.09 0)
+		(effects
+			(font
+				(size 1.27 1.27)
+			)
+			(justify left)
 		)
 	)
@@
 		(shape input)
 		(at 162.56 92.71 0)
+		(effects
+			(font
+				(size 1.27 1.27)
+			)
+			(justify left)
+		)
+	)
+	(hierarchical_label "ACCEL_2.5V_POWER_SENSITIVE"
+		(shape input)
+		(at 185.42 82.55 0)
 		(effects
 			(font
@@
 	)
 	(symbol
-		(lib_id "power:+3.3V")
-		(at 185.42 85.09 270)
-		(unit 1)
-		(exclude_from_sim no)
-		(in_bom yes)
-		(on_board yes)
-		(dnp no)
-		(fields_autoplaced yes)
-		(property "Reference" "#PWR027"
-			(at 181.61 85.09 0)
-			(effects
-				(font
-					(size 1.27 1.27)
-				)
-				(hide yes)
-			)
-		)
-		(property "Value" "+3.3V"
-			(at 189.23 85.0899 90)
-			(effects
-				(font
-					(size 1.27 1.27)
-				)
-				(justify left)
-			)
-		)
-		(property "Footprint" ""
-			(at 185.42 85.09 0)
-			(effects
-				(font
-					(size 1.27 1.27)
-				)
-				(hide yes)
-			)
-		)
-		(property "Datasheet" ""
-			(at 185.42 85.09 0)
-			(effects
-				(font
-					(size 1.27 1.27)
-				)
-				(hide yes)
-			)
-		)
-		(property "Description" "Power symbol creates a global label with name \"+3.3V\""
-			(at 185.42 85.09 0)
-			(effects
-				(font
-					(size 1.27 1.27)
-				)
-				(hide yes)
-			)
-		)
-		(pin "1"
-		)
-		(instances
-			(project "SRAD FC Rev B"
-				(path "/1dd9e63a-24f2-43c6-ae21-66b89e6998f2/a64879cb-ca83-46f5-8e0d-bba02df69177"
-					(reference "#PWR027")
-					(unit 1)
-				)
-			)
-		)
-	)
-	(symbol
 		(lib_id "Device:C_Small")
 		(at 179.07 74.93 0)
@@
 					(unit 1)
 				)
-			)
-		)
-	)
-	(symbol
-		(lib_id "power:+3.3V")
-		(at 185.42 82.55 270)
-		(unit 1)
-		(exclude_from_sim no)
-		(in_bom yes)
-		(on_board yes)
-		(dnp no)
-		(fields_autoplaced yes)
-		(property "Reference" "#PWR026"
-			(at 181.61 82.55 0)
-			(effects
-				(font
-					(size 1.27 1.27)
-				)
-				(hide yes)
-			)
-		)
-		(property "Value" "+2.5V"
-			(at 189.23 82.5499 90)
-			(effects
-				(font
-					(size 1.27 1.27)
-				)
-				(justify left)
-			)
-		)
-		(property "Footprint" ""
-			(at 185.42 82.55 0)
-			(effects
-				(font
-					(size 1.27 1.27)
-				)
-				(hide yes)
-			)
-		)
-		(property "Datasheet" ""
-			(at 185.42 82.55 0)
-			(effects
-				(font
-					(size 1.27 1.27)
-				)
-				(hide yes)
-			)
-		)
-		(property "Description" "Power symbol creates a global label with name \"+1.8V\""
-			(at 185.42 82.55 0)
-			(effects
-				(font
-					(size 1.27 1.27)
-				)
-				(hide yes)
-			)
-		)
-		(pin "1"
-		)
-		(instances
-			(project "SRAD FC Rev B"
-				(path "/1dd9e63a-24f2-43c6-ae21-66b89e6998f2/a64879cb-ca83-46f5-8e0d-bba02df69177"
-					(reference "#PWR026")
-					(unit 1)
-				)

Commit message: fixed some library symbold
Parts:
- U2: footprint ADXL372BCCZ-RL7:PQFN50P322X300X114-16N -> ADXL372BCCZ_RL7:PQFN50P322X300X114-16N
Changed lines of the file:
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@@
 			)
 		)
-		(property "Footprint" "ADXL372BCCZ-RL7:PQFN50P322X300X114-16N"
+		(property "Footprint" "ADXL372BCCZ_RL7:PQFN50P322X300X114-16N"
 			(at 144.78 92.71 0)
 			(effects

Commit message: set up power conversion, wired power to mcu
Parts:
- removed U2: ADXL372BCCZ-RL7, ADXL372BCCZ_RL7:PQFN50P322X300X114-16N, symbol ADXL372BCCZ-RL7:ADXL372BCCZ-RL7
- added U6: ADXL372BCCZ-RL7, ADXL372BCCZ-RL7:PQFN50P322X300X114-16N, symbol ADXL372BCCZ-RL7:ADXL372BCCZ-RL7
Connections:
- net ACCEL_2.5V_POWER_SENSITIVE: now also U6.14 (VS)
- net ACCEL_3.3V_POWER: now also U6.1 (VDDI/O)
- net ACCEL_INT1: now also U6.11 (INT1)
- net ACCEL_INT2: now also U6.9 (INT2)
- net ACCEL_SPI_CS: now also U6.8 (~{CS}/SCL)
- net ACCEL_SPI_MISO: now also U6.7 (MISO)
- net ACCEL_SPI_MOSI: now also U6.6 (MOSI/SDA)
- net ACCEL_SPI_SCLK: now also U6.4 (SCLK)
- net GND: now also U6.12 (GND), U6.13 (GND__1), U6.16 (GND__2)
Changed lines of the file:
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@@
-	)
-	(symbol
-		(lib_id "ADXL372BCCZ-RL7:ADXL372BCCZ-RL7")
-		(at 144.78 92.71 0)
-		(unit 1)
-		(exclude_from_sim no)
-		(in_bom yes)
-		(on_board yes)
-		(dnp no)
-		(fields_autoplaced yes)
-		(property "Reference" "U2"
-			(at 144.78 74.93 0)
-			(effects
-				(font
-					(size 1.27 1.27)
-				)
-			)
-		)
-		(property "Value" "ADXL372BCCZ-RL7"
-			(at 144.78 77.47 0)
-			(effects
-				(font
-					(size 1.27 1.27)
-				)
-			)
-		)
-		(property "Footprint" "ADXL372BCCZ_RL7:PQFN50P322X300X114-16N"
-			(at 144.78 92.71 0)
-			(effects
-				(font
-					(size 1.27 1.27)
-				)
-				(justify bottom)
-				(hide yes)
-			)
-		)
-		(property "Datasheet" ""
-			(at 144.78 92.71 0)
-			(effects
-				(font
-					(size 1.27 1.27)
-				)
-				(hide yes)
-			)
-		)
-		(property "Description" ""
-			(at 144.78 92.71 0)
-			(effects
-				(font
-					(size 1.27 1.27)
-				)
-				(hide yes)
-			)
-		)
-		(property "PARTREV" "B"
-			(at 144.78 92.71 0)
-			(effects
-				(font
-					(size 1.27 1.27)
-				)
-				(justify bottom)
-				(hide yes)
-			)
-		)
-		(property "STANDARD" "IPC-7351B"
-			(at 144.78 92.71 0)
-			(effects
-				(font
-					(size 1.27 1.27)
-				)
-				(justify bottom)
-				(hide yes)
-			)
-		)
-		(property "MANUFACTURER" "Analog Devices"
-			(at 144.78 92.71 0)
-			(effects
-				(font
-					(size 1.27 1.27)
-				)
-				(justify bottom)
-				(hide yes)
-			)
-		)
-		(pin "13"
-		)
-		(pin "9"
-		)
-		(pin "16"
-		)
-		(pin "11"
-		)
-		(pin "1"
-		)
-		(pin "7"
-		)
-		(pin "14"
-		)
-		(pin "6"
-		)
-		(pin "4"
-		)
-		(pin "12"
-		)
-		(pin "8"
-		)
-		(instances
-			(project ""
-				(path "/1dd9e63a-24f2-43c6-ae21-66b89e6998f2/a64879cb-ca83-46f5-8e0d-bba02df69177"
-					(reference "U2")
-					(unit 1)
-				)
-			)
-		)
 	)
 	(symbol
@@
 					(unit 1)
 				)
+			)
+		)
+	)
+	(symbol
+		(lib_id "ADXL372BCCZ-RL7:ADXL372BCCZ-RL7")
+		(at 144.78 92.71 0)
+		(unit 1)
+		(exclude_from_sim no)
+		(in_bom yes)
+		(on_board yes)
+		(dnp no)
+		(fields_autoplaced yes)
+		(property "Reference" "U6"
+			(at 144.78 74.93 0)
+			(effects
+				(font
+					(size 1.27 1.27)
+				)
+			)
+		)
+		(property "Value" "ADXL372BCCZ-RL7"
+			(at 144.78 77.47 0)
+			(effects
+				(font
+					(size 1.27 1.27)
+				)
+			)
+		)
+		(property "Footprint" "ADXL372BCCZ-RL7:PQFN50P322X300X114-16N"
+			(at 144.78 92.71 0)
+			(effects
+				(font
+					(size 1.27 1.27)
+				)
+				(justify bottom)
+				(hide yes)
+			)
+		)
+		(property "Datasheet" ""
+			(at 144.78 92.71 0)
+			(effects
+				(font
+					(size 1.27 1.27)
+				)
+				(hide yes)
+			)
+		)
+		(property "Description" ""
+			(at 144.78 92.71 0)
+			(effects
+				(font
+					(size 1.27 1.27)
+				)
+				(hide yes)
+			)
+		)
+		(property "PARTREV" "B"
+			(at 144.78 92.71 0)
+			(effects
+				(font
+					(size 1.27 1.27)
+				)
+				(justify bottom)
+				(hide yes)
+			)
+		)
+		(property "STANDARD" "IPC-7351B"
+			(at 144.78 92.71 0)
+			(effects
+				(font
+					(size 1.27 1.27)
+				)
+				(justify bottom)
+				(hide yes)
+			)
+		)
+		(property "MANUFACTURER" "Analog Devices"
+			(at 144.78 92.71 0)
+			(effects
+				(font
+					(size 1.27 1.27)
+				)
+				(justify bottom)
+				(hide yes)
+			)
+		)
+		(pin "13"
+		)
+		(pin "14"
+		)
+		(pin "8"
+		)
+		(pin "6"
+		)
+		(pin "4"
+		)
+		(pin "9"
+		)
+		(pin "7"
+		)
+		(pin "1"
+		)
+		(pin "11"
+		)
+		(pin "12"
+		)
+		(pin "16"
+		)
+		(instances
+			(project ""
+				(path "/1dd9e63a-24f2-43c6-ae21-66b89e6998f2/a64879cb-ca83-46f5-8e0d-bba02df69177"
+					(reference "U6")
+					(unit 1)
+				)
